File: pi_PCB_2.0/pi_PCB_2.0.kicad_pcb (KiCad board)
At the start: 2 copper layers, 160 x 90 mm, 7 parts

Commit message: PCB Final?
Parts:
- moved Raspberry_Pi1 2.04 mm to (87.7, 97.0)
- moved Screen_and_Sensor_Header1 1.04 mm to (177.5, 112.0)
Connections:
- Motors_Header1 pad 1: Net-(Motors_Header1-3V3_Power-Pad1) -> Net-(Line_Sensor_Holes1-VCC)
- Motors_Header1 pad 17: Net-(Line_Sensor_Holes1-VCC) -> Net-(Motors_Header1-3V3_Power-Pad17)
- Motors_Header1 pad 20: Net-(Motors_Header1-Ground-Pad20) -> Net-(Motors_Header1-Ground-Pad14)
- Motors_Header1 pad 25: Net-(Motors_Header1-Ground-Pad25) -> Net-(Motors_Header1-Ground-Pad14)
- Motors_Header1 pad 6: Net-(Motors_Header1-Ground-Pad6) -> Net-(Motors_Header1-Ground-Pad14)
- Motors_Header1 pad 9: Net-(Motors_Header1-Ground-Pad9) -> Net-(Motors_Header1-Ground-Pad14)
- Raspberry_Pi1 pad 1: Net-(Motors_Header1-3V3_Power-Pad1) -> Net-(Line_Sensor_Holes1-VCC)
- Raspberry_Pi1 pad 17: Net-(Line_Sensor_Holes1-VCC) -> Net-(Motors_Header1-3V3_Power-Pad17)
- Raspberry_Pi1 pad 20: Net-(Motors_Header1-Ground-Pad20) -> Net-(Motors_Header1-Ground-Pad14)
- Raspberry_Pi1 pad 25: Net-(Motors_Header1-Ground-Pad25) -> Net-(Motors_Header1-Ground-Pad14)
- Raspberry_Pi1 pad 6: Net-(Motors_Header1-Ground-Pad6) -> Net-(Motors_Header1-Ground-Pad14)
- Raspberry_Pi1 pad 9: Net-(Motors_Header1-Ground-Pad9) -> Net-(Motors_Header1-Ground-Pad14)
- Screen_and_Sensor_Header1 pad 1: Net-(Motors_Header1-3V3_Power-Pad1) -> Net-(Line_Sensor_Holes1-VCC)
- Screen_and_Sensor_Header1 pad 17: Net-(Line_Sensor_Holes1-VCC) -> Net-(Motors_Header1-3V3_Power-Pad17)
- Screen_and_Sensor_Header1 pad 20: Net-(Motors_Header1-Ground-Pad20) -> Net-(Motors_Header1-Ground-Pad14)
- Screen_and_Sensor_Header1 pad 25: Net-(Motors_Header1-Ground-Pad25) -> Net-(Motors_Header1-Ground-Pad14)
- Screen_and_Sensor_Header1 pad 6: Net-(Motors_Header1-Ground-Pad6) -> Net-(Motors_Header1-Ground-Pad14)
- Screen_and_Sensor_Header1 pad 9: Net-(Motors_Header1-Ground-Pad9) -> Net-(Motors_Header1-Ground-Pad14)
Routing:
- net Net-(Motors_Header1-3V3_Power-Pad1): track 200.3 -> 0.00 mm
- net Net-(Motors_Header1-Ground-Pad20): track 193.5 -> 0.00 mm
- net Net-(Motors_Header1-3V3_Power-Pad17): track 0.00 -> 153.1 mm
- net Net-(Motors_Header1-5V_Power-Pad4): track 0.00 -> 139.1 mm
- net Net-(Motors_Header1-Ground-Pad14): track 95.8 -> 215.3 mm
- net Net-(Line_Sensor_Holes1-Ground): track 29.1 -> 89.4 mm
- net Net-(Line_Sensor_Holes1-VCC): track 256.3 -> 203.2 mm
- net Net-(Motors_Header1-GPIO_21): track 0.00 -> 52.6 mm
- net Net-(Motors_Header1-Ground-Pad25): track 33.2 -> 0.00 mm
- net Net-(Line_Sensor_Holes1-Out): track 62.8 -> 72.1 mm
- net Net-(Raspberry_Pi1-SDA/GPIO2): track 95.1 -> 100.3 mm
- net Net-(Motors_Header1-GPIO_14): track 124.4 -> 129.4 mm
- net Net-(Raspberry_Pi1-SCL/GPIO3): track 95.7 -> 100.6 mm
- net Net-(Ultrasonic_Holes1-VCC): track 144.4 -> 148.4 mm
- net Net-(Raspberry_Pi1-GPIO25): track 96.2 -> 99.4 mm
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- added copper zone on F.Cu, net Net-(Motors_Header1-Ground-Pad14)
Other:
- outline, holes or cut-outs redrawn

Commit message: Final 2
Parts:
- added REF**: MountingHole_2.5mm, MountingHole:MountingHole_2.5mm, F.Cu at (224.0, 85.0)
- added REF**: MountingHole_2.5mm, MountingHole:MountingHole_2.5mm, F.Cu at (224.0, 154.0)
- added REF**: MountingHole_2.5mm, MountingHole:MountingHole_2.5mm, F.Cu at (90.5, 85.0)
- moved Raspberry_Pi1 14.1 mm to (96.7, 86.0)
- moved Ultrasonic_Holes1 3.04 mm to (81.0, 100.0)
- moved Line_Sensor_Holes1 2.50 mm to (84.0, 79.5)
- moved 330_Resistor1 1.58 mm to (82.5, 88.5)
- moved 470_Resistor1 1.58 mm to (82.5, 85.5)
Routing:
- net Net-(Motors_Header1-Ground-Pad14): track 215.3 -> 51.7 mm
- net Net-(Raspberry_Pi1-GCLK1/GPIO5): track 49.8 -> 86.5 mm
- net Net-(Line_Sensor_Holes1-VCC): track 203.2 -> 177.2 mm
- net Net-(Motors_Header1-GPIO_14): track 129.4 -> 114.4 mm
- net Net-(Motors_Header1-5V_Power-Pad4): track 139.1 -> 124.9 mm
- net Net-(Motors_Header1-GPIO_15): track 121.3 -> 111.0 mm
- net Net-(Raspberry_Pi1-GCLK2/GPIO6): track 49.5 -> 59.2 mm
- net Net-(Line_Sensor_Holes1-Out): track 72.1 -> 64.3 mm
- net Net-(Motors_Header1-GPIO_13): track 73.5 -> 66.4 mm
- net Net-(Raspberry_Pi1-GPIO25): track 99.4 -> 92.6 mm
- net Net-(Motors_Header1-GPIO_19): track 67.6 -> 61.0 mm
- net Net-(Motors_Header1-GPIO_20): track 59.7 -> 54.6 mm
- net Net-(Raspberry_Pi1-GPIO17): track 99.2 -> 94.1 mm
- net Net-(Line_Sensor_Holes1-Ground): track 89.4 -> 94.2 mm
- net Net-(Raspberry_Pi1-~{CE0}/GPIO8): track 97.1 -> 92.6 mm
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Other:
- outline, holes or cut-outs redrawn

Commit message: Final 3
Parts:
- removed 330_Resistor1, 470_Resistor1: R_Small, Resistor_THT:R_Axial_DIN0204_L3.6mm_D1.6mm_P1.90mm_Vertical
- added 330: R_Small, Resistor_THT:R_Axial_DIN0207_L6.3mm_D2.5mm_P10.16mm_Horizontal, F.Cu at (86.5, 100.2)
- added 470: R_Small, Resistor_THT:R_Axial_DIN0207_L6.3mm_D2.5mm_P10.16mm_Horizontal, F.Cu at (90.5, 100.2)
- Raspberry_Pi1: value Raspberry_Pi_2_3 -> Power
- Screen_and_Sensor_Header1: value Screen_and_Sensor_Header -> Screen_and_Sensor
- renumbered Line_Sensor_Holes1 to Line_Sensor, Motors_Header1 to Motors, Ultrasonic_Holes1 to Ultrasonic
Connections:
- Line_Sensor pad 1: Net-(Line_Sensor_Holes1-VCC) -> Net-(Line_Sensor_Holes1-Ground)
- Line_Sensor pad 2: Net-(Line_Sensor_Holes1-Ground) -> Net-(Line_Sensor_Holes1-VCC)
Routing:
- net Net-(Motors_Header1-Ground-Pad14): track 51.7 -> 96.8 mm
- net Net-(Line_Sensor_Holes1-VCC): track 177.2 -> 218.9 mm
- net Net-(Ultrasonic_Holes1-VCC): track 149.5 -> 167.7 mm
- net Net-(Raspberry_Pi1-GCLK2/GPIO6): track 59.2 -> 66.7 mm
- net Net-(Raspberry_Pi1-GCLK1/GPIO5): track 86.5 -> 80.6 mm
- net Net-(Line_Sensor_Holes1-Ground): track 94.2 -> 92.4 mm
Other:
- outline, holes or cut-outs redrawn
- board text added: "Screen & Sensors"
